Commit message: Car URDF almost done, just need to put the sensors (gyroscope and lidar)

File: urdf_ws/src/urdfbot_description/urdf/urdfbot_simple.urdf (robot description, URDF)
Before this commit: robot urdfbot, 1 links, 0 joints
Links:
- removed link base_link
- added link body_link; visual box size=0.256 0.150 0.065
- added link wheel1_link; visual cylinder length=0.025 radius=0.033
- added link wheel2_link; visual cylinder length=0.025 radius=0.033
- added link wheel3_link; visual cylinder length=0.025 radius=0.033
- added link wheel4_link; visual cylinder length=0.025 radius=0.033
Joints:
- added joint wheel1_joint: type fixed, parent body_link, child wheel1_link, origin xyz=-0.0575 -0.0665 -0.03, axis 0 0 0
- added joint wheel2_joint: type fixed, parent body_link, child wheel2_link, origin xyz=-0.0575 0.0665 -0.03, axis 0 0 0
- added joint wheel3_joint: type fixed, parent body_link, child wheel3_link, origin xyz=0.0575 0.0665 -0.03, axis 0 0 0
- added joint wheel4_joint: type fixed, parent body_link, child wheel4_link, origin xyz=0.0575 -0.0665 -0.03, axis 0 0 0

Commit message: URDF model of our testing car for NAV is finished

File: urdf_ws/src/urdfbot_description/urdf/urdfbot_simple.urdf (robot description, URDF)
Before this commit: robot urdfbot, 5 links, 4 joints
Links:
- added link gyro_link; visual box size=0.02 0.02 0.015
- added link lidarB_link; visual box size=0.08 0.08 0.005
- added link lidar_link; visual box size=0.05 0.05 0.030
- added link struct1_link; visual box size=0.01 0.01 0.038
- added link struct2_link; visual box size=0.01 0.01 0.038
- added link struct3_link; visual box size=0.01 0.01 0.038
Joints:
- added joint gyro_joint: type fixed, parent body_link, child gyro_link, origin xyz=-0.03 0.0 0.0325, axis 0 0 0
- added joint lidarB_joint: type fixed, parent struct1_link, child lidarB_link, origin xyz=-0.03 0.0 0.019, axis 0 0 0
- added joint lidar_joint: type fixed, parent lidarB_link, child lidar_link, origin xyz=0.0 0.0 0.013, axis 0 0 0
- added joint struct1_joint: type fixed, parent body_link, child struct1_link, origin xyz=0.0 0.0 0.05, axis 0 0 0
- added joint struct2_joint: type fixed, parent body_link, child struct2_link, origin xyz=-0.059 0.0115 0.05, axis 0 0 0
- added joint struct3_joint: type fixed, parent body_link, child struct3_link, origin xyz=-0.059 -0.0115 0.05, axis 0 0 0
- joint wheel4_joint: axis 0 0 0 -> 0 0 1
